File: PiRadio/PiRadio.sch (KiCad schematic (older format))
At the start: 69 parts, among them P1 SMA_female, P2 SMA_female, T1 ETC1-1-13, U1 HMC599, U2 HMC432, U3 ADL5387

Commit message: changes of CompLib & Shem
add ADcon
Parts:
- added C43: 2700p, symbol C
- added C44: 0.047u, symbol C
- added C45: 680p, symbol C
- added C46, C47, C48, C62, C63, C64, C65: 0.1u, symbol C
- added C49, C50: 10u, symbol C
- added C51, C52, C56, C57: 220p, symbol C
- added C53, C54: 470p, symbol C
- added C55, C58, C59, C60, C61: C, symbol C
- added D2: Led_Small, symbol Led_Small
- added L10, L11, L12, L13, L14, L15, L16, L9: 820n, symbol L_Small
- added P3: CONN_02X20, symbol CONN_02X20
- added R11, R16, R17, R28, R29, R31, R32: R, symbol R
- added R12: 360, symbol R
- added R13, R30, R33, R34, R35: 0, symbol R
- added R14: 1k, symbol R
- added R15, R18, R19: 100, symbol R
- added R20, R21, R22, R23: 470, symbol R
- added R24, R25, R26, R27: 4.7k, symbol R
- added U5: AD9218, symbol AD9218
- added U6, U7: ADA4940, symbol ADA4940
- gave numbers to parts that had none: 37
Connections:
- net 5V: now also C49.1, C50.1, P3.27 (P27)
- net A3V: now also C20.1, C47.1, C48.1, C58.1, C59.1, C60.1, C61.1, C63.1, C65.1, R16.1, U5.15 (V_DD), U5.28 (V_DD), U5.33 (V_DD), U5.46 (V_DD), U6.3 (+Vs), U7.3 (+Vs)
- net GNDA: now also C43.2, C45.2, C49.2, C50.2, C55.2, C58.2, C59.2, C60.2, C61.2, C63.2, C65.2, D2.1 (K), R13.2, R17.2, R34.1, R35.1, U5.1 (GND), U5.12 (GND), U6.6 (-Vs), U7.6 (-Vs)
- net IH: now also C52.1, L11.1
- net IL: now also C52.2, L12.2
- net PLL_CK: now also P3.35 (P35)
- net PLL_DA: now also P3.37 (P37)
- net PLL_LE: now also P3.39 (P39)
- net QH: now also C51.1, L9.1
- net QL: now also C51.2, L10.2
- net at U4.20 (V_TUNE): now also C45.1, R14.1
- net at U4.25 (LD): now also R15.2
- net at U4.5 (SW): now also R11.1
- net at U4.7 (CP_OUT): now also C43.1, C44.1, R14.2
- new net: C44.2, R12.2
- new net: R11.2, R12.1, R13.1
- new net: D2.2 (A), R15.1
- new net: R26.1, U5.10 (AinBn), U7.5 (OUT-)
- new net: R27.1, U5.11 (AinBp), U7.4 (OUT+)
- new net: R25.1, U5.2 (AinAp), U6.4 (OUT+)
- new net: R24.1, U5.3 (AinAn), U6.5 (OUT-)
- new net: R28.1, R29.1, U5.4 (DFS/GAIN)
- new net: U5.5 (REFinA), U5.6 (REFout), U5.7 (REFinB)
- new net: R30.1, R31.1, U5.8 (S1)
- new net: R32.1, R33.1, U5.9 (S2)
- new net: R21.1, R25.2, U6.1 (IN-)
- new net: C55.1, R16.2, R17.1, U6.2 (Vcom), U7.2 (Vcom)
- new net: R20.1, R24.2, U6.8 (IN+)
- new net: C56.2, L14.1, R18.2, R21.2
- new net: C56.1, L13.2, R18.1, R20.2
- new net: C53.1, L13.1, L9.2
- new net: C53.2, L10.1, L14.2
- new net: R23.1, R27.2, U7.1 (IN-)
- new net: R22.1, R26.2, U7.8 (IN+)
- new net: C57.2, L16.1, R19.2, R23.2
- new net: C57.1, L15.2, R19.1, R22.2
- new net: C54.1, L11.2, L15.1
- new net: C54.2, L12.1, L16.2
- new net 3V: C46.1, C62.1, C64.1, R28.2, R30.2, R32.2, U5.13 (V_D), U5.30 (V_D), U5.31 (V_D), U5.48 (V_D)
- new net DI0: P3.2 (P2), U5.35 (D0A)
- new net DI1: P3.4 (P4), U5.36 (D1A)
- new net DI2: P3.5 (P5), U5.37 (D2A)
- new net DI3: P3.6 (P6), U5.38 (D3A)
- new net DI4: P3.7 (P7), U5.39 (D4A)
- new net DI5: P3.8 (P8), U5.40 (D5A)
- new net DI6: P3.9 (P9), U5.41 (D6A)
- new net DI7: P3.10 (P10), U5.42 (D7A)
- new net DI8: P3.13 (P13), U5.43 (D8A)
- new net DI9: P3.14 (P14), U5.44 (D9A)
- new net DQ0: P3.15 (P15), U5.26 (D0B)
- new net DQ1: P3.16 (P16), U5.25 (D1B)
- new net DQ2: P3.17 (P17), U5.24 (D2B)
- new net DQ3: P3.18 (P18), U5.23 (D3B)
- new net DQ4: P3.19 (P19), U5.22 (D4B)
- new net DQ5: P3.20 (P20), U5.21 (D5B)
- new net DQ6: P3.21 (P21), U5.20 (D6B)
- new net DQ7: P3.22 (P22), U5.19 (D7B)
- new net DQ8: P3.23 (P23), U5.18 (D8B)
- new net DQ9: P3.24 (P24), U5.17 (D9B)
- new net ENCA: P3.25 (P25), U5.47 (ENCa)
- new net ENCB: P3.26 (P26), U5.14 (ENCb)
- new net GNDD: C46.2, C47.2, C48.2, C62.2, C64.2, P3.29 (P29), R29.2, R31.2, R33.2, R34.2, R35.2, U5.16 (GND), U5.27 (GND), U5.29 (GND), U5.32 (GND), U5.34 (GND), U5.45 (GND)
- no-connect marks 1 -> 17
Other:
- moved on the sheet: C25, C26
