File: PiRadio/PiRadio.sch (KiCad schematic (older format))
At the start: 136 parts, among them P1 SMA_female, P2 SMA_female, P3 CONN_02X20, T1 ETC1-1-13, U1 HMC599, U2 HMC432, U3 ADL5387, U4 ADF4351, U5 AD9218, U6 ADA4940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

Commit message: changes of pcb
route and patern completed
Parts:
- U4: footprint Housings_DFN_QFN:QFN-32-1EP_5x5mm_Pitch0.5mm -> MyLibrary:QFN-32-1EP_5x5mm_Pitch0.5mm
Connections:
- net GNDA: now also U2.2 (GND)
Changed lines of the file:
@@
 L GNDA #PWR06
 U 1 1 585CE07D
-P 6250 2950
-F 0 "#PWR06" H 6250 2700 50  0001 C CNN
-F 1 "GNDA" H 6250 2800 50  0000 C CNN
-F 2 "" H 6250 2950 50  0000 C CNN
-F 3 "" H 6250 2950 50  0000 C CNN
-	1    6250 2950
+P 3050 3500
+F 0 "#PWR06" H 3050 3250 50  0001 C CNN
+F 1 "GNDA" H 3050 3350 50  0000 C CNN
+F 2 "" H 3050 3500 50  0000 C CNN
+F 3 "" H 3050 3500 50  0000 C CNN
+	1    3050 3500
 	1    0    0    -1
 $EndComp
@@
 F 0 "U4" H 3150 5950 60  0000 C CNN
 F 1 "ADF4351" H 3700 5050 60  0000 C CNN
-F 2 "Housings_DFN_QFN:QFN-32-1EP_5x5mm_Pitch0.5mm" H 3700 5300 60  0001 C CNN
+F 2 "MyLibrary:QFN-32-1EP_5x5mm_Pitch0.5mm" H 3700 5300 60  0001 C CNN
 F 3 "" H 3700 5300 60  0000 C CNN
 	1    3700 5300
