File: PiRadio/PiRadio.kicad_pcb (KiCad board)
At the start: 2 copper layers, 66.5 x 77.7 mm, 142 parts, among them P1 SMA_female, P2 SMA_female, P3 CONN_02X20, T1 ETC1-1-13, U1 HMC599, U2 HMC432, U3 ADL5387, U4 ADF4351, U5 AD9218, U6 ADA4940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

Commit message: changes of pcb
route and patern completed
Parts:
- removed REF** (x3): QFN-24_4x4mm_Pitch0.5mm_NoMask, MyLibrary:QFN-24_4x4mm_Pitch0.5mm_SarmalPad
- removed the U4 at (0.00, 0.00) (x3)
- C29, C30, C43, R11: moved to F.Cu
- C33, C34: moved to B.Cu
- U4: footprint Housings_DFN_QFN:QFN-32-1EP_5x5mm_Pitch0.5mm -> MyLibrary:QFN-32-1EP_5x5mm_Pitch0.5mm
- moved R34 3.56 mm to (133.6, 118.4)
- moved C30 2.88 mm to (90.0, 90.9)
- moved C29 2.53 mm to (90.0, 92.5)
- moved C33 1.63 mm to (89.9, 88.9)
- moved C34 1.55 mm to (89.9, 87.4)
- moved R10 1.02 mm to (88.8, 94.5)
- moved C17 1.02 mm to (102.6, 91.9)
- moved C18 1.02 mm to (102.6, 94.0)
- moved C64 0.95 mm to (130.0, 121.9)
- moved C65 0.95 mm to (130.0, 124.0)
- moved L6 0.64 mm to (86.4, 88.9)
- moved C31 0.07 mm to (89.0, 93.5)
Connections:
- U2 pad 2: Net-(U2-Pad2) -> GNDA
Routing:
- net GNDA: track 3.12 -> 456.2 mm, vias 0 -> 2
- net A3V: track 70.9 -> 271.1 mm, vias 7 -> 8
- net GNDD: track 0.00 -> 161.5 mm, vias 0 -> 2
- net 5V: track 6.57 -> 141.9 mm, vias 0 -> 2
- net (no net): track 118.9 -> 0.00 mm, vias 5 -> 4
- net PLL_CK: track 0.00 -> 104.3 mm
- net PLL_DA: track 0.00 -> 94.9 mm
- net PLL_LE: track 0.00 -> 84.6 mm, vias 0 -> 1
- net DI0: track 0.00 -> 62.7 mm, vias 0 -> 1
- net DQ9: track 0.00 -> 52.3 mm
- net DI1: track 0.00 -> 49.6 mm
- net DQ7: track 0.00 -> 49.3 mm
- net 3V: track 11.4 -> 60.6 mm, vias 0 -> 1
- net DI5: track 0.00 -> 49.2 mm, vias 0 -> 1
- net DI7: track 0.00 -> 49.0 mm
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- added copper zone on B.Cu, net GNDA
